Commit message: Added MQ2 lib and code refactoring
Added MQ2 lib, changed <> to "", adjusted indents and made small code refactoring.

File: RPi_motor_interface/urdf/robot.urdf.xacro (robot description, xacro)
@@ -1,100 +1,100 @@
 <?xml version="1.0"?>
 <robot xmlns:xacro="http://ros.org/wiki/xacro" name="robot_description">
-  <!-- Material -->
-  <material name="white">
-    <color rgba="1 1 1 1"/>
-  </material>
-  <material name="gray">
-    <color rgba="0.6 0.6 0.6 1"/>
-  </material>
-  <material name="black">
-    <color rgba="0 0 0 1"/>
-  </material>
-  <!-- Base link -->
-  <link name="base_link">
-    <visual>
-      <geometry>
-        <box size="0.18 0.13 0.05"/>
-      </geometry>
-      <material name="gray"/>
-    </visual>
-    <collision>
-      <geometry>
-        <box size="0.18 0.13 0.05"/>
-      </geometry>
-    </collision>
-    <inertial>
-      <mass value="1.0"/>
-      <inertia ixx="0.01" ixy="0.0" ixz="0.0" iyy="0.01" iyz="0.0" izz="0.01"/>
-    </inertial>
-  </link>
+	<!-- Material -->
+	<material name="white">
+		<color rgba="1 1 1 1"/>
+	</material>
+	<material name="gray">
+		<color rgba="0.6 0.6 0.6 1"/>
+	</material>
+	<material name="black">
+		<color rgba="0 0 0 1"/>
+	</material>
+	<!-- Base link -->
+	<link name="base_link">
+		<visual>
+			<geometry>
+			<box size="0.18 0.13 0.05"/>
+			</geometry>
+			<material name="gray"/>
+		</visual>
+		<collision>
+			<geometry>
+			<box size="0.18 0.13 0.05"/>
+			</geometry>
+		</collision>
+		<inertial>
+			<mass value="1.0"/>
+			<inertia ixx="0.01" ixy="0.0" ixz="0.0" iyy="0.01" iyz="0.0" izz="0.01"/>
+		</inertial>
+	</link>
   <!-- Base footprint for SLAM -->
-  <link name="base_footprint" />
-  <joint name="base_footprint_to_base_link" type="fixed">
-    <parent link="base_footprint"/>
-    <child link="base_link"/>
-    <origin xyz="0 0 0.3" rpy="0 0 0"/>
-  </joint>
+	<link name="base_footprint" />
+	<joint name="base_footprint_to_base_link" type="fixed">
+		<parent link="base_footprint"/>
+		<child link="base_link"/>
+		<origin xyz="0 0 0.3" rpy="0 0 0"/>
+	</joint>
   <!-- Wheels -->
-  <link name="wheel_left">
-    <visual>
-      <geometry>
-        <cylinder radius="0.035" length="0.02"/>
-      </geometry>
-      <origin xyz="0 0 0" rpy="1.5708 0 0"/>
-      <material name="black"/>
-    </visual>
-  </link>
-  <link name="wheel_right">
-    <visual>
-      <geometry>
-        <cylinder radius="0.035" length="0.02"/>
-      </geometry>
-      <origin xyz="0 0 0" rpy="1.5708 0 0"/>
-      <material name="black"/>
-    </visual>
-  </link>
-  <!-- Joints for wheels -->
-  <joint name="left_wheel_joint" type="continuous">
-    <parent link="base_link"/>
-    <child link="wheel_left"/>
-    <origin xyz="0 -0.10 0" rpy="0 0 0"/>
-    <axis xyz="0 1 0"/>
-  </joint>
-  <joint name="right_wheel_joint" type="continuous">
-    <parent link="base_link"/>
-    <child link="wheel_right"/>
-    <origin xyz="0 0.10 0" rpy="0 0 0"/>
-    <axis xyz="0 1 0"/>
-  </joint>
-  <!-- LIDAR -->
-  <link name="laser">
-    <visual>
-      <geometry>
-        <cylinder radius="0.03" length="0.02"/>
-      </geometry>
-      <origin xyz="0.06 0 0.10" rpy="0 0 0"/>
-      <material name="gray"/>
-    </visual>
-  </link>
-  <joint name="laser_joint" type="fixed">
-    <parent link="base_link"/>
-    <child link="laser"/>
-    <origin xyz="0.06 0 0.10" rpy="0 0 3.1416"/>   <!-- obrót o pi=180 stopni -->
-  </joint>
-  <!-- Ultrasonic sensor -->
-  <link name="ultrasonic_link">
-    <visual>
-      <geometry>
-        <box size="0.03 0.01 0.01"/>
-      </geometry>
-      <origin xyz="0.09 0 0.025" rpy="0 0 0"/>
-      <material name="gray"/>
-    </visual>
-  </link>
-  <joint name="ultrasonic_joint" type="fixed">
-    <parent link="base_link"/>
-    <child link="ultrasonic_link"/>
-    <origin xyz="0.09 0 0.025" rpy="0 0 0"/>
-  </joint>
+	<link name="wheel_left">
+		<visual>
+			<geometry>
+			<cylinder radius="0.035" length="0.02"/>
+			</geometry>
+			<origin xyz="0 0 0" rpy="1.5708 0 0"/>
+			<material name="black"/>
+		</visual>
+	</link>
+	<link name="wheel_right">
+		<visual>
+			<geometry>
+			<cylinder radius="0.035" length="0.02"/>
+			</geometry>
+			<origin xyz="0 0 0" rpy="1.5708 0 0"/>
+			<material name="black"/>
+		</visual>
+	</link>
+	<!-- Joints for wheels -->
+	<joint name="left_wheel_joint" type="continuous">
+		<parent link="base_link"/>
+		<child link="wheel_left"/>
+		<origin xyz="0 -0.10 0" rpy="0 0 0"/>
+		<axis xyz="0 1 0"/>
+	</joint>
+	<joint name="right_wheel_joint" type="continuous">
+		<parent link="base_link"/>
+		<child link="wheel_right"/>
+		<origin xyz="0 0.10 0" rpy="0 0 0"/>
+		<axis xyz="0 1 0"/>
+	</joint>
+	<!-- LIDAR -->
+	<link name="laser">
+		<visual>
+			<geometry>
+			<cylinder radius="0.03" length="0.02"/>
+			</geometry>
+			<origin xyz="0.06 0 0.10" rpy="0 0 0"/>
+			<material name="gray"/>
+		</visual>
+	</link>
+	<joint name="laser_joint" type="fixed">
+		<parent link="base_link"/>
+		<child link="laser"/>
+		<origin xyz="0.06 0 0.10" rpy="0 0 3.1416"/>   <!-- obrót o pi=180 stopni -->
+	</joint>
+	<!-- Ultrasonic sensor -->
+	<link name="ultrasonic_link">
+		<visual>
+			<geometry>
+			<box size="0.03 0.01 0.01"/>
+			</geometry>
+			<origin xyz="0.09 0 0.025" rpy="0 0 0"/>
+			<material name="gray"/>
+		</visual>
+	</link>
+	<joint name="ultrasonic_joint" type="fixed">
+		<parent link="base_link"/>
+		<child link="ultrasonic_link"/>
+		<origin xyz="0.09 0 0.025" rpy="0 0 0"/>
+	</joint>
 </robot>
